File: pcb/polymod3/Module1.sch (KiCad schematic (older format))
At the start: 21 parts

Commit message: pcb layout (early)
Parts:
- C1: renamed from C?; footprint (none) -> Capacitor_THT:CP_Radial_D5.0mm_P2.50mm
- J2, J3: renamed from J?; footprint (none) -> Connector_PinHeader_2.54mm:PinHeader_1x08_P2.54mm_Vertical
- R1, R10, R11, R12, R13, R14, R15, R16, R2, R3, R4, R5, R6, R7, R8, R9: renamed from R?; footprint (none) -> Resistor_THT:R_Axial_DIN0207_L6.3mm_D2.5mm_P7.62mm_Horizontal
- U3, U4: renamed from U?; footprint (none) -> Package_DIP:DIP-16_W7.62mm_Socket
Connections:
- net GND: now also U3.13 (~OE)
- net VCC: now also U3.10 (~SRCLR)

Commit message: still playing in kicad
Parts:
- removed C1: 10uF, Capacitor_THT:CP_Radial_D5.0mm_P2.50mm, symbol Device:CP
- added D1, D2, D3, D4: LED, LED_THT:LED_D5.0mm, symbol Device:LED
- added R17, R18, R19, R20: R, Resistor_THT:R_Axial_DIN0207_L6.3mm_D2.5mm_P7.62mm_Horizontal, symbol Device:R
- added RV1, RV2, RV3, RV4: R_POT, Potentiometer_THT:Potentiometer_Alps_RK09K_Single_Vertical, symbol Device:R_POT
- added U2: 74HC595, Package_DIP:DIP-16_W7.62mm_Socket, symbol 74xx:74HC595
- added U5: 4051, Package_DIP:DIP-16_W7.62mm_Socket, symbol 4xxx:4051
Connections:
- no-connect marks 1 -> 61

Commit message: nice
Parts:
- R17, R18, R19, R20: value R -> 680
Connections:
- net GND: now also D1.1 (K), D2.1 (K), D3.1 (K), D4.1 (K), RV1.3, RV2.3, RV3.3, RV4.3, U2.13 (~OE), U2.8 (GND), U5.6 (Inh), U5.7 (VEE), U5.8 (VSS)
- net VCC: now also RV1.1, RV2.1, RV3.1, RV4.1, U2.10 (~SRCLR), U2.16 (VCC), U5.16 (VDD)
- net POT1: now reaches RV1.2
- net POT1: now also U5.13 (X0)
- net at U2.1 (QB): now also R18.2
- net LED_CLOCK: now reaches U2.11 (SRCLK)
- net LED_LATCH: now reaches U2.12 (RCLK)
- net LED_DATA_IN: now reaches U2.14 (SER)
- net at U2.15 (QA): now also R17.2
- net at U2.2 (QC): now also R19.2
- net at U2.3 (QD): now also R20.2
- net LED_DATA_OUT: now reaches U2.9 (QH')
- net ANA_CHAN1: now reaches U5.10 (B)
- net ANA_CHAN0: now reaches U5.11 (A)
- net POT4: now reaches U5.12 (X3)
- net POT4: now also RV4.2
- net POT2: now reaches U5.14 (X1)
- net POT2: now also RV2.2
- net POT3: now reaches U5.15 (X2)
- net POT3: now also RV3.2
- net ANA_OUT: now reaches U5.3 (X)
- net ANA_CHAN2: now reaches U5.9 (C)
- net at D1.2 (A): now also R17.1
- net at D3.2 (A): now also R19.1
- net at D2.2 (A): now also R18.1
- net at D4.2 (A): now also R20.1
- no-connect marks 61 -> 9
Other:
- note added: "LEDs"
- note added: "Potentiometers"
- moved on the sheet: D1, D2, D3, D4, R17, R18, R19, R20, RV1, RV2, RV3, RV4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
