File: pcb/polymod3/polymod3.sch (KiCad schematic (older format))
At the start: 6 parts

Commit message: kicad stuff
Parts:
- removed U? (x4): 74HC595, symbol 74xx:74HC595
- removed U?: 4051, symbol 4xxx:4051
- added DIS?: HD44780, 16026-16X2, symbol HD44780:HD44780
- added J?: DIN-5_180degree, symbol Connector:DIN-5_180degree
- added U?: 6N138, symbol Isolator:6N138
Connections:
- net VCC: now reaches U?.51 (3V3)
- net GND: now reaches U?.52 (GND)
- no-connect marks 0 -> 16
Other:
- note removed: "Analog controls"
- note removed: "Input shift registers"
- note removed: "Output shift registers"
Changed lines of the file:
@@
 $Descr A3 16535 11693
 encoding utf-8
-Sheet 1 1
+Sheet 1 2
 Title ""
 Date ""
@@
 	1    0    0    -1
 $EndComp
+$Sheet
+S 10500 3400 2100 1400
+U 60216398
+F0 "Module1" 50
+F1 "Module1.sch" 50
+$EndSheet
 $Comp
-L 74xx:74HC595 U?
-U 1 1 60108BB0
-P 2850 2200
-F 0 "U?" H 2850 2981 50  0000 C CNN
-F 1 "74HC595" H 2850 2890 50  0000 C CNN
-F 2 "" H 2850 2200 50  0001 C CNN
-F 3 "http://www.ti.com/lit/ds/symlink/sn74hc595.pdf" H 2850 2200 50  0001 C CNN
-	1    2850 2200
+L Connector:DIN-5_180degree J?
+U 1 1 60225E90
+P 12200 2100
+F 0 "J?" H 12200 1825 50  0000 C CNN
+F 1 "DIN-5_180degree" H 12200 1734 50  0000 C CNN
+F 2 "" H 12200 2100 50  0001 C CNN
+F 3 "http://www.mouser.com/ds/2/18/40_c091_abd_e-75918.pdf" H 12200 2100 50  0001 C CNN
+	1    12200 2100
 	1    0    0    -1
 $EndComp
 $Comp
-L 74xx:74HC595 U?
-U 1 1 601095F2
-P 4200 2200
-F 0 "U?" H 4200 2981 50  0000 C CNN
-F 1 "74HC595" H 4200 2890 50  0000 C CNN
-F 2 "" H 4200 2200 50  0001 C CNN
-F 3 "http://www.ti.com/lit/ds/symlink/sn74hc595.pdf" H 4200 2200 50  0001 C CNN
-	1    4200 2200
-	1    0    0    -1
-$EndComp
-Text Notes 3100 1100 0    50   ~ 0
-Output shift registers
-$Comp
-L 74xx:74HC595 U?
-U 1 1 6010CD70
-P 2850 4650
-F 0 "U?" H 2850 5431 50  0000 C CNN
-F 1 "74HC595" H 2850 5340 50  0000 C CNN
-F 2 "" H 2850 4650 50  0001 C CNN
-F 3 "http://www.ti.com/lit/ds/symlink/sn74hc595.pdf" H 2850 4650 50  0001 C CNN
-	1    2850 4650
+L Isolator:6N138 U?
+U 1 1 60226C14
+P 10450 2200
+F 0 "U?" H 10450 2667 50  0000 C CNN
+F 1 "6N138" H 10450 2576 50  0000 C CNN
+F 2 "" H 10740 1900 50  0001 C CNN
+F 3 "http://www.onsemi.com/pub/Collateral/HCPL2731-D.pdf" H 10740 1900 50  0001 C CNN
+	1    10450 2200
 	1    0    0    -1
 $EndComp
 $Comp
-L 74xx:74HC595 U?
-U 1 1 6010CD76
-P 4200 4650
-F 0 "U?" H 4200 5431 50  0000 C CNN
-F 1 "74HC595" H 4200 5340 50  0000 C CNN
-F 2 "" H 4200 4650 50  0001 C CNN
-F 3 "http://www.ti.com/lit/ds/symlink/sn74hc595.pdf" H 4200 4650 50  0001 C CNN
-	1    4200 4650
+L HD44780:HD44780 DIS?
+U 1 1 602278FC
+P 3550 1900
+F 0 "DIS?" H 4080 896 50  0000 L CNN
+F 1 "HD44780" H 4080 805 50  0000 L CNN
+F 2 "16026-16X2" H 3550 1900 50  0001 L BNN
+F 3 "" H 3550 1900 50  0001 L BNN
+F 4 "5V" H 3550 1900 50  0001 L BNN "VOLTAGE"
+F 5 "N/A" H 3550 1900 50  0001 L BNN "MGF#"
+	1    3550 1900
 	1    0    0    -1
 $EndComp
-Text Notes 3100 3550 0    50   ~ 0
-Input shift registers
 $Comp
-L 4xxx:4051 U?
-U 1 1 6010D122
-P 12050 2400
-F 0 "U?" H 12594 2446 50  0000 L CNN
-F 1 "4051" H 12594 2355 50  0000 L CNN
-F 2 "" H 12050 2400 50  0001 C CNN
-F 3 "http://www.intersil.com/content/dam/Intersil/documents/cd40/cd4051bms-52bms-53bms.pdf" H 12050 2400 50  0001 C CNN
-	1    12050 2400
+L power:VCC #PWR?
+U 1 1 6023FEF3
+P 8000 7750
+F 0 "#PWR?" H 8000 7600 50  0001 C CNN
+F 1 "VCC" H 8015 7923 50  0000 C CNN
+F 2 "" H 8000 7750 50  0001 C CNN
+F 3 "" H 8000 7750 50  0001 C CNN
+	1    8000 7750
 	1    0    0    -1
 $EndComp
-Text Notes 11850 1150 0    50   ~ 0
-Analog controls
+NoConn ~ 8000 7400
+NoConn ~ 8450 7400
+NoConn ~ 8600 7400
+NoConn ~ 9400 7000
+NoConn ~ 9400 6900
+NoConn ~ 9400 6800
+NoConn ~ 9400 6700
+NoConn ~ 9400 6600
+NoConn ~ 9400 6500
+NoConn ~ 7200 7100
+NoConn ~ 7200 7000
+NoConn ~ 7200 6900
+NoConn ~ 7200 6800
+NoConn ~ 7200 6700
+NoConn ~ 7200 6550
+NoConn ~ 7200 6450
+Wire Wire Line
+	8000 7750 8150 7750
+Wire Wire Line
+	8150 7750 8150 7400
+$Comp
+L power:GND #PWR?
+U 1 1 60241B6E
+P 8300 7400
+F 0 "#PWR?" H 8300 7150 50  0001 C CNN
+F 1 "GND" H 8305 7227 50  0000 C CNN
+F 2 "" H 8300 7400 50  0001 C CNN
+F 3 "" H 8300 7400 50  0001 C CNN
+	1    8300 7400
+	1    0    0    -1
+$EndComp
 $EndSCHEMATC

Commit message: pcb layout (early)
Parts:
- removed DIS?: HD44780, 16026-16X2, symbol HD44780:HD44780
- removed J?: DIN-5_180degree, symbol Connector:DIN-5_180degree
- removed U?: 6N138, symbol Isolator:6N138
- U1: renamed from U?; footprint (none) -> teensy:Teensy41
Connections:
- net GND: now also U1.1 (GND), U1.34 (GND), U1.47 (GND); no longer U1.52 (GND)
- net VCC: now also U1.15 (3V3); no longer U1.51 (3V3)
- net IN_LOAD: now reaches U1.10 (8_TX2_IN1)
- net IN_CLOCK_ENABLE: now reaches U1.11 (9_OUT1C)
- net IN_CLOCK: now reaches U1.12 (10_CS_MQSR)
- net Module1/IN_DATA_OUT: now reaches U1.13 (11_MOSI_CTX1)
- net OUT_CLOCK: now reaches U1.38 (16_A2_RX4_SCL1)
- net OUT_LATCH: now reaches U1.39 (17_A3_TX4_SDA1)
- net Module1/OUT_DATA_IN: now reaches U1.44 (22_A8_CTX1)
- no-connect marks 16 -> 58
Changed lines of the file:
@@
 $EndDescr
 $Comp
-L teensy:Teensy4.1 U?
+L teensy:Teensy4.1 U1
 U 1 1 6010669C
 P 8300 6100
-F 0 "U?" H 8300 8665 50  0000 C CNN
+F 0 "U1" H 8300 8665 50  0000 C CNN
 F 1 "Teensy4.1" H 8300 8574 50  0000 C CNN
-F 2 "" H 7900 6500 50  0001 C CNN
+F 2 "teensy:Teensy41" H 7900 6500 50  0001 C CNN
 F 3 "" H 7900 6500 50  0001 C CNN
 	1    8300 6100
@@
 $EndComp
 $Sheet
-S 10500 3400 2100 1400
+S 10650 4500 2100 1400
 U 60216398
 F0 "Module1" 50
 F1 "Module1.sch" 50
+F2 "OUT_DATA_IN" I L 10650 4750 50
+F3 "OUT_DATA_OUT" O L 10650 4900 50
+F4 "IN_DATA_OUT" O L 10650 5450 50
+F5 "IN_DATA_IN" I L 10650 5300 50
 $EndSheet
-$Comp
-L Connector:DIN-5_180degree J?
-U 1 1 60225E90
-P 12200 2100
-F 0 "J?" H 12200 1825 50  0000 C CNN
-F 1 "DIN-5_180degree" H 12200 1734 50  0000 C CNN
-F 2 "" H 12200 2100 50  0001 C CNN
-F 3 "http://www.mouser.com/ds/2/18/40_c091_abd_e-75918.pdf" H 12200 2100 50  0001 C CNN
-	1    12200 2100
-	1    0    0    -1
-$EndComp
-$Comp
-L Isolator:6N138 U?
-U 1 1 60226C14
-P 10450 2200
-F 0 "U?" H 10450 2667 50  0000 C CNN
-F 1 "6N138" H 10450 2576 50  0000 C CNN
-F 2 "" H 10740 1900 50  0001 C CNN
-F 3 "http://www.onsemi.com/pub/Collateral/HCPL2731-D.pdf" H 10740 1900 50  0001 C CNN
-	1    10450 2200
-	1    0    0    -1
-$EndComp
-$Comp
-L HD44780:HD44780 DIS?
-U 1 1 602278FC
-P 3550 1900
-F 0 "DIS?" H 4080 896 50  0000 L CNN
-F 1 "HD44780" H 4080 805 50  0000 L CNN
-F 2 "16026-16X2" H 3550 1900 50  0001 L BNN
-F 3 "" H 3550 1900 50  0001 L BNN
-F 4 "5V" H 3550 1900 50  0001 L BNN "VOLTAGE"
-F 5 "N/A" H 3550 1900 50  0001 L BNN "MGF#"
-	1    3550 1900
-	1    0    0    -1
-$EndComp
-$Comp
-L power:VCC #PWR?
-U 1 1 6023FEF3
-P 8000 7750
-F 0 "#PWR?" H 8000 7600 50  0001 C CNN
-F 1 "VCC" H 8015 7923 50  0000 C CNN
-F 2 "" H 8000 7750 50  0001 C CNN
-F 3 "" H 8000 7750 50  0001 C CNN
-	1    8000 7750
-	1    0    0    -1
-$EndComp
 NoConn ~ 8000 7400
 NoConn ~ 8450 7400
@@
 NoConn ~ 7200 6550
 NoConn ~ 7200 6450
+NoConn ~ 9400 3800
+NoConn ~ 9400 3950
+NoConn ~ 8300 7400
+NoConn ~ 8150 7400
+$Comp
+L power:GND #PWR0101
+U 1 1 6024265D
+P 7200 3950
+F 0 "#PWR0101" H 7200 3700 50  0001 C CNN
+F 1 "GND" V 7205 3822 50  0000 R CNN
+F 2 "" H 7200 3950 50  0001 C CNN
+F 3 "" H 7200 3950 50  0001 C CNN
+	1    7200 3950
+	0    1    1    0
+$EndComp
+$Comp
+L power:GND #PWR0102
+U 1 1 60242A46
+P 9400 5350
+F 0 "#PWR0102" H 9400 5100 50  0001 C CNN
+F 1 "GND" V 9405 5222 50  0000 R CNN
+F 2 "" H 9400 5350 50  0001 C CNN
+F 3 "" H 9400 5350 50  0001 C CNN
+	1    9400 5350
+	0    -1   -1   0
+$EndComp
+$Comp
+L power:VCC #PWR0103
+U 1 1 602437FE
+P 6850 5350
+F 0 "#PWR0103" H 6850 5200 50  0001 C CNN
+F 1 "VCC" V 6865 5477 50  0000 L CNN
+F 2 "" H 6850 5350 50  0001 C CNN
+F 3 "" H 6850 5350 50  0001 C CNN
+	1    6850 5350
+	0    -1   -1   0
+$EndComp
+NoConn ~ 9400 4150
+$Comp
+L power:GND #PWR0104
+U 1 1 602441A9
+P 9400 4050
+F 0 "#PWR0104" H 9400 3800 50  0001 C CNN
+F 1 "GND" V 9405 3922 50  0000 R CNN
+F 2 "" H 9400 4050 50  0001 C CNN
+F 3 "" H 9400 4050 50  0001 C CNN
+	1    9400 4050
+	0    -1   -1   0
+$EndComp
+Text GLabel 9400 4850 2    50   Output ~ 0
+OUT_LATCH
+Text GLabel 9400 4950 2    50   Output ~ 0
+OUT_CLOCK
+Text GLabel 7200 4850 0    50   Output ~ 0
+IN_LOAD
+Text GLabel 7200 4950 0    50   Output ~ 0
+IN_CLOCK_ENABLE
+Text GLabel 7200 5050 0    50   Output ~ 0
+IN_CLOCK
+NoConn ~ 7200 4650
+NoConn ~ 7200 4750
+NoConn ~ 9400 4750
+NoConn ~ 9400 4650
+NoConn ~ 9400 4550
+NoConn ~ 9400 4450
+NoConn ~ 9400 4250
+NoConn ~ 7200 4050
+NoConn ~ 7200 4150
+NoConn ~ 7200 4250
+NoConn ~ 7200 4350
+NoConn ~ 7200 4450
+NoConn ~ 7200 4550
+NoConn ~ 7200 5250
+NoConn ~ 7200 5450
+NoConn ~ 7200 5550
+NoConn ~ 7200 5650
+NoConn ~ 7200 5750
+NoConn ~ 7200 5850
+NoConn ~ 7200 5950
+NoConn ~ 7200 6050
+NoConn ~ 7200 6150
+NoConn ~ 7200 6250
+NoConn ~ 9400 6250
+NoConn ~ 9400 6150
+NoConn ~ 9400 6050
+NoConn ~ 9400 5950
+NoConn ~ 9400 5850
+NoConn ~ 9400 5750
+NoConn ~ 9400 5650
+NoConn ~ 9400 5550
+NoConn ~ 9400 5450
+NoConn ~ 9400 5250
+NoConn ~ 9400 5150
+NoConn ~ 9400 5050
 Wire Wire Line
-	8000 7750 8150 7750
+	9400 4350 10250 4350
 Wire Wire Line
-	8150 7750 8150 7400
+	10250 4350 10250 4750
+Wire Wire Line
+	10250 4750 10650 4750
+Wire Wire Line
+	7200 5150 6150 5150
+Wire Wire Line
+	6150 5150 6150 7550
+Wire Wire Line
+	6150 7550 10250 7550
+Wire Wire Line
+	10250 7550 10250 5450
+Wire Wire Line
+	10250 5450 10650 5450
+NoConn ~ 10650 5300
+NoConn ~ 10650 4900
+Wire Wire Line
+	7200 5350 6900 5350
 $Comp
-L power:GND #PWR?
-U 1 1 60241B6E
-P 8300 7400
-F 0 "#PWR?" H 8300 7150 50  0001 C CNN
-F 1 "GND" H 8305 7227 50  0000 C CNN
-F 2 "" H 8300 7400 50  0001 C CNN
-F 3 "" H 8300 7400 50  0001 C CNN
-	1    8300 7400
-	1    0    0    -1
+L power:PWR_FLAG #FLG0101
+U 1 1 6024B298
+P 6900 5350
+F 0 "#FLG0101" H 6900 5425 50  0001 C CNN
+F 1 "PWR_FLAG" H 6900 5523 50  0000 C CNN
+F 2 "" H 6900 5350 50  0001 C CNN
+F 3 "~" H 6900 5350 50  0001 C CNN
+	1    6900 5350
+	-1   0    0    1
 $EndComp
+Connection ~ 6900 5350
+Wire Wire Line
+	6900 5350 6850 5350
 $EndSCHEMATC

Commit message: nice
Parts:
- added H1, H2, H3, H4, H5, H6: MountingHole, MountingHole:MountingHole_3.2mm_M3, symbol Mechanical:MountingHole
- added U6: 4051, Package_DIP:DIP-16_W7.62mm_Socket, symbol 4xxx:4051
Connections:
- net GND: now also U6.6 (Inh), U6.7 (VEE), U6.8 (VSS)
- net VCC: now also U6.16 (VDD)
- net ANA_MAIN: now reaches U1.14 (12_MISO_MQSL)
- net ANA_MAIN: now also U6.3 (X)
- net ANA_CHAN0: now reaches U1.2 (0_RX1_CRX2_CS1)
- net ANA_CHAN1: now reaches U1.3 (1_TX1_CTX2_MISO1)
- net ANA_CHAN2: now reaches U1.4 (2_OUT2)
- net ANA_MAIN_CHAN0: now reaches U1.5 (3_LRCLK2)
- net ANA_MAIN_CHAN0: now also U6.11 (A)
- net ANA_MAIN_CHAN1: now reaches U1.6 (4_BCLK2)
- net ANA_MAIN_CHAN1: now also U6.10 (B)
- net ANA_MAIN_CHAN2: now reaches U1.7 (5_IN2)
- net ANA_MAIN_CHAN2: now also U6.9 (C)
- net LED_CLOCK: now reaches U1.8 (6_OUT1D)
- net LED_LATCH: now reaches U1.9 (7_RX2_OUT1A)
- new net Module1/ANA_OUT: U6.13 (X0)
Other:
- moved on the sheet: U1
