File: pcb/polymod3/polymod3.kicad_pcb (KiCad board)
At the start: 2 copper layers, 250 x 110 mm, 22 parts, among them J2 Conn_01x08_Female, J3 Conn_01x08_Female, U1 Teensy4.1, U3 74HC595, U4 74HC165

Commit message: still playing in kicad
Parts:
- removed C1: 10uF, Capacitor_THT:CP_Radial_D5.0mm_P2.50mm
- added D1: LED, LED_THT:LED_D5.0mm, F.Cu at (53.3, 50.8)
- added D2: LED, LED_THT:LED_D5.0mm, F.Cu at (53.3, 35.6)
- added D3: LED, LED_THT:LED_D5.0mm, F.Cu at (53.3, 66.0)
- added D4: LED, LED_THT:LED_D5.0mm, F.Cu at (53.3, 81.3)
- added H1: MountingHole, MountingHole:MountingHole_3.2mm_M3, F.Cu at (47.0, 35.0)
- added H2: MountingHole, MountingHole:MountingHole_3.2mm_M3, F.Cu at (57.0, 135.0)
- added H3: MountingHole, MountingHole:MountingHole_3.2mm_M3, F.Cu at (-30.1, 68.6)
- added H4: MountingHole, MountingHole:MountingHole_3.2mm_M3, F.Cu at (-30.1, 76.5)
- added H5: MountingHole, MountingHole:MountingHole_3.2mm_M3, F.Cu at (-22.2, 68.6)
- added H6: MountingHole, MountingHole:MountingHole_3.2mm_M3, F.Cu at (-22.2, 76.5)
- added R17: R, Resistor_THT:R_Axial_DIN0207_L6.3mm_D2.5mm_P7.62mm_Horizontal, F.Cu at (50.8, 43.2)
- added R18: R, Resistor_THT:R_Axial_DIN0207_L6.3mm_D2.5mm_P7.62mm_Horizontal, F.Cu at (50.8, 58.4)
- added R19: R, Resistor_THT:R_Axial_DIN0207_L6.3mm_D2.5mm_P7.62mm_Horizontal, F.Cu at (50.8, 73.7)
- added R20: R, Resistor_THT:R_Axial_DIN0207_L6.3mm_D2.5mm_P7.62mm_Horizontal, F.Cu at (50.8, 88.9)
- added RV1: R_POT, Potentiometer_THT:Potentiometer_Alps_RK09K_Single_Vertical, F.Cu at (30.5, 43.2)
- added RV2: R_POT, Potentiometer_THT:Potentiometer_Alps_RK09K_Single_Vertical, F.Cu at (30.5, 88.9)
- added RV3: R_POT, Potentiometer_THT:Potentiometer_Alps_RK09K_Single_Vertical, F.Cu at (30.5, 73.7)
- added RV4: R_POT, Potentiometer_THT:Potentiometer_Alps_RK09K_Single_Vertical, F.Cu at (30.5, 58.4)
- added U2: 74HC595, Package_DIP:DIP-16_W7.62mm_Socket, B.Cu at (45.7, 66.0)
- added U5: 4051, Package_DIP:DIP-16_W7.62mm_Socket, B.Cu at (45.7, 40.6)
- moved R11 63.3 mm to (27.9, 99.1)
- moved R13 55.9 mm to (27.9, 104.1)
- moved R12 53.0 mm to (27.9, 101.6)
- moved R9 49.1 mm to (27.9, 94.0)
- moved R15 44.7 mm to (27.9, 109.2)
- moved R14 34.1 mm to (27.9, 106.7)
- moved R16 31.5 mm to (27.9, 111.8)
- moved R10 23.0 mm to (27.9, 96.5)
- moved U3 21.6 mm to (50.8, 116.8), turned to 180 degrees
- moved U4 13.7 mm to (43.2, 111.8), turned to 0 degrees
- moved J2 2.54 mm to (22.9, 116.8)
- moved J3 2.54 mm to (22.9, 94.0)
- moved R1 2.54 mm to (27.9, 116.8)
- moved R2 2.54 mm to (27.9, 119.4)
- moved R3 2.54 mm to (27.9, 121.9)
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
Commit message: nice
Parts:
- added U6: 4051, Package_DIP:DIP-16_W7.62mm_Socket, B.Cu at (250.0, 129.0)
- R17, R18, R19, R20: value R -> 680
Connections:
- net Net-(U2-Pad14) renamed /Module1/LED_DATA_IN
- net Net-(U2-Pad9) renamed /Module1/LED_DATA_OUT
- D1 pad 1: Net-(D1-Pad1) -> GND
- D2 pad 1: Net-(D2-Pad1) -> GND
- D3 pad 1: Net-(D3-Pad1) -> GND
- D4 pad 1: Net-(D4-Pad1) -> GND
- R17 pad 1: Net-(R17-Pad1) -> Net-(D1-Pad2)
- R18 pad 1: Net-(R18-Pad1) -> Net-(D2-Pad2)
- R19 pad 1: Net-(R19-Pad1) -> Net-(D3-Pad2)
- R20 pad 1: Net-(R20-Pad1) -> Net-(D4-Pad2)
- RV1 pad 1: Net-(RV1-Pad1) -> VCC
- RV1 pad 2: Net-(RV1-Pad2) -> /Module1/POT1
- RV1 pad 3: Net-(RV1-Pad3) -> GND
- RV2 pad 1: Net-(RV2-Pad1) -> VCC
- RV2 pad 2: Net-(RV2-Pad2) -> /Module1/POT2
- RV2 pad 3: Net-(RV2-Pad3) -> GND
- RV3 pad 1: Net-(RV3-Pad1) -> VCC
- RV3 pad 2: Net-(RV3-Pad2) -> /Module1/POT3
- RV3 pad 3: Net-(RV3-Pad3) -> GND
- RV4 pad 1: Net-(RV4-Pad1) -> VCC
- RV4 pad 2: Net-(RV4-Pad2) -> /Module1/POT4
- RV4 pad 3: Net-(RV4-Pad3) -> GND
- U1 pad 14: Net-(U1-Pad14) -> /ANA_MAIN
- U1 pad 2: Net-(U1-Pad2) -> ANA_CHAN0
- U1 pad 3: Net-(U1-Pad3) -> ANA_CHAN1
- U1 pad 4: Net-(U1-Pad4) -> ANA_CHAN2
- U1 pad 5: Net-(U1-Pad5) -> /ANA_MAIN_CHAN0
- U1 pad 6: Net-(U1-Pad6) -> /ANA_MAIN_CHAN1
- U1 pad 7: Net-(U1-Pad7) -> /ANA_MAIN_CHAN2
- U1 pad 8: Net-(U1-Pad8) -> LED_CLOCK
- U1 pad 9: Net-(U1-Pad9) -> LED_LATCH
- U2 pad 1: Net-(U2-Pad1) -> Net-(R18-Pad2)
- U2 pad 10: Net-(U2-Pad10) -> VCC
- U2 pad 11: Net-(U2-Pad11) -> LED_CLOCK
- U2 pad 12: Net-(U2-Pad12) -> LED_LATCH
- U2 pad 13: Net-(U2-Pad13) -> GND
- U2 pad 15: Net-(U2-Pad15) -> Net-(R17-Pad2)
- U2 pad 16: Net-(U2-Pad16) -> VCC
- U2 pad 2: Net-(U2-Pad2) -> Net-(R19-Pad2)
- U2 pad 3: Net-(U2-Pad3) -> Net-(R20-Pad2)
- U2 pad 8: Net-(U2-Pad8) -> GND
- U5 pad 10: Net-(U5-Pad10) -> ANA_CHAN1
- U5 pad 11: Net-(U5-Pad11) -> ANA_CHAN0
- U5 pad 12: Net-(U5-Pad12) -> /Module1/POT4
- U5 pad 13: Net-(U5-Pad13) -> /Module1/POT1
- U5 pad 14: Net-(U5-Pad14) -> /Module1/POT2
- U5 pad 15: Net-(U5-Pad15) -> /Module1/POT3
- U5 pad 16: Net-(U5-Pad16) -> VCC
- U5 pad 3: Net-(U5-Pad3) -> /Module1/ANA_OUT
- U5 pad 6: Net-(U5-Pad6) -> GND
- U5 pad 7: Net-(U5-Pad7) -> GND
- U5 pad 8: Net-(U5-Pad8) -> GND
- U5 pad 9: Net-(U5-Pad9) -> ANA_CHAN2

Commit message: routing...
Parts:
- moved RV2 30.5 mm to (30.5, 58.4)
- moved RV4 30.5 mm to (30.5, 88.9)
- moved D1 15.2 mm to (53.3, 35.6)
- moved D2 15.2 mm to (53.3, 50.8)
- moved H2 3.00 mm to (57.0, 132.0)
Routing:
- net VCC: track 0.00 -> 144.2 mm
- net /Module1/POT4: track 0.00 -> 43.7 mm
- net Net-(J3-Pad8): track 0.00 -> 36.9 mm
- net /Module1/POT3: track 0.00 -> 36.2 mm
- net Net-(R17-Pad2): track 0.00 -> 34.4 mm
- net Net-(J3-Pad7): track 0.00 -> 31.2 mm
- net Net-(J3-Pad4): track 0.00 -> 30.0 mm
- net Net-(J3-Pad3): track 0.00 -> 30.0 mm
- net Net-(J3-Pad2): track 0.00 -> 30.0 mm
- net Net-(J3-Pad1): track 0.00 -> 30.0 mm
- net Net-(R20-Pad2): track 0.00 -> 29.4 mm
- net Net-(J3-Pad6): track 0.00 -> 25.7 mm
- net /Module1/POT1: track 0.00 -> 21.6 mm
- net Net-(J3-Pad5): track 0.00 -> 21.4 mm
- net /Module1/POT2: track 0.00 -> 18.9 mm
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- added copper zone on B.Cu, net GND
- added copper zone on F.Cu, net GND

Commit message: about to change the design again...
Parts:
- moved R1 121.9 mm to (149.9, 118.1)
- moved R10 121.9 mm to (149.9, 97.8)
- moved R11 121.9 mm to (149.9, 100.3)
- moved R12 121.9 mm to (149.9, 102.9)
- moved R13 121.9 mm to (149.9, 105.4)
- moved R14 121.9 mm to (149.9, 108.0)
- moved R15 121.9 mm to (149.9, 110.5)
- moved R16 121.9 mm to (149.9, 113.0)
- moved R2 121.9 mm to (149.9, 120.7)
- moved R3 121.9 mm to (149.9, 123.2)
- moved R4 121.9 mm to (149.9, 125.7)
- moved R5 121.9 mm to (149.9, 128.3)
- moved R6 121.9 mm to (149.9, 130.8)
- moved R7 121.9 mm to (149.9, 133.3)
- moved R8 121.9 mm to (149.9, 135.9)
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