File: pcb/p3mini/p3mini.kicad_pcb (KiCad board)
At the start: 2 copper layers, 100 x 100 mm, 104 parts, among them J1 Conn_02x12_Odd_Even, J2 Conn_02x12_Odd_Even, J3 DIN-5_180degree, J4 Conn_01x10, U1 74HC595, U10 4051, U11 4051, U2 74HC595, U3 74HC595, U4 74HC165, U5 74HC165, U6 74HC165, U7 74HC595, U8 Teensy4.1, U9 6N138

Commit message: layout
Parts:
- C1, D9, J3, J4, R1, R10, R11, R12, R13, R14, R15, R16, R17, R18, R19, R2, R20, R21, R22, R23, R24, R25, R26, R27, R28, R29, R3, R30, R31, R32, R33, R34, R35, R36, R37, R38, R39, R4, R40, R41, R42, R43, R44, R45, R46, R47, R48, R49, R5, R50, R51, R52, R53, R54, R55, R56, R57, R58, R59, R6, R7, R8, R9, U1, U10, U11, U2, U3, U4, U5, U6, U7, U8, U9: moved to B.Cu
- moved R52 170.1 mm to (12.7, 70.0), turned to 270 degrees
- moved D9 167.8 mm to (112.7, 5.08)
- moved R53 163.2 mm to (15.2, 64.9), turned to 270 degrees
- moved R20 160.4 mm to (34.6, 76.2), turned to 180 degrees
- moved U10 159.8 mm to (40.0, 21.0), turned to 270 degrees
- moved R19 159.1 mm to (34.6, 78.7), turned to 180 degrees
- moved R24 158.5 mm to (34.6, 66.0), turned to 180 degrees
- moved R22 151.5 mm to (34.6, 71.1), turned to 180 degrees
- moved R3 151.3 mm to (44.1, 71.1)
- moved R5 151.2 mm to (44.1, 76.2)
- moved R16 148.5 mm to (34.6, 86.4), turned to 180 degrees
- moved R2 146.9 mm to (44.1, 68.6)
- moved R17 146.5 mm to (34.6, 83.8), turned to 180 degrees
- moved R15 146.2 mm to (34.6, 88.9), turned to 180 degrees
- moved R1 145.5 mm to (44.1, 66.0)
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- renumbered RV11 to RV10, RV14 to RV11, RV16 to RV12, RV3 to RV13, RV6 to RV14, RV9 to RV15, RV12 to RV16, RV4 to RV2, RV7 to RV3, RV10 to RV4, RV13 to RV5, RV15 to RV6, RV2 to RV7, RV5 to RV8, RV8 to RV9
Connections:
- J1 pad 10: /OUTPUT9 -> /OUTPUT19
- J1 pad 11: /OUTPUT10 -> /OUTPUT5
- J1 pad 12: /OUTPUT11 -> /OUTPUT18
- J1 pad 13: /OUTPUT12 -> /OUTPUT6
- J1 pad 14: /OUTPUT13 -> /OUTPUT17
- J1 pad 15: /OUTPUT14 -> /OUTPUT7
- J1 pad 16: /OUTPUT15 -> /OUTPUT16
- J1 pad 17: /OUTPUT16 -> /OUTPUT8
- J1 pad 18: /OUTPUT17 -> /OUTPUT15
- J1 pad 19: /OUTPUT18 -> /OUTPUT9
- J1 pad 2: /OUTPUT1 -> /OUTPUT23
- J1 pad 20: /OUTPUT19 -> /OUTPUT14
- J1 pad 21: /OUTPUT20 -> /OUTPUT10
- J1 pad 22: /OUTPUT21 -> /OUTPUT13
- J1 pad 23: /OUTPUT22 -> /OUTPUT11
- J1 pad 24: /OUTPUT23 -> /OUTPUT12
- J1 pad 3: /OUTPUT2 -> /OUTPUT1
- J1 pad 4: /OUTPUT3 -> /OUTPUT22
- J1 pad 5: /OUTPUT4 -> /OUTPUT2
- J1 pad 6: /OUTPUT5 -> /OUTPUT21
- J1 pad 7: /OUTPUT6 -> /OUTPUT3
- J1 pad 8: /OUTPUT7 -> /OUTPUT20
- J1 pad 9: /OUTPUT8 -> /OUTPUT4
- J2 pad 10: /INPUT9 -> /INPUT19
- J2 pad 11: /INPUT10 -> /INPUT5
- J2 pad 12: /INPUT11 -> /INPUT18
- J2 pad 13: /INPUT12 -> /INPUT6
- J2 pad 14: /INPUT13 -> /INPUT17
- J2 pad 15: /INPUT14 -> /INPUT7
- J2 pad 16: /INPUT15 -> /INPUT16
- J2 pad 17: /INPUT16 -> /INPUT8
- J2 pad 18: /INPUT17 -> /INPUT15
- J2 pad 19: /INPUT18 -> /INPUT9
- J2 pad 2: /INPUT1 -> /INPUT23
- J2 pad 20: /INPUT19 -> /INPUT14
- J2 pad 21: /INPUT20 -> /INPUT10
- J2 pad 22: /INPUT21 -> /INPUT13
- J2 pad 23: /INPUT22 -> /INPUT11
- J2 pad 24: /INPUT23 -> /INPUT12
- J2 pad 3: /INPUT2 -> /INPUT1
- J2 pad 4: /INPUT3 -> /INPUT22
- J2 pad 5: /INPUT4 -> /INPUT2
- J2 pad 6: /INPUT5 -> /INPUT21
- J2 pad 7: /INPUT6 -> /INPUT3
- J2 pad 8: /INPUT7 -> /INPUT20
- J2 pad 9: /INPUT8 -> /INPUT4
Other:
- board size 100 x 100 mm -> 140 x 100 mm
