File: pcb/p3mini/p3mini.sch (KiCad schematic (older format))
At the start: 73 parts, among them J2 Conn_02x10_Odd_Even, U1 74HC595, U2 74HC165, U3 74HC595, U4 4051

Commit message: polymod mini looks good so far
Parts:
- removed J2: Conn_02x10_Odd_Even, Connector_PinHeader_2.54mm:PinHeader_2x10_P2.54mm_Vertical, symbol Connector_Generic:Conn_02x10_Odd_Even
- added D? (x4): LED, LED_THT:LED_D5.0mm, symbol Device:LED
- added H? (x2): MountingHole, MountingHole:MountingHole_3.2mm_M3, symbol Mechanical:MountingHole
- added R? (x4): 220, Resistor_SMD:R_1206_3216Metric, symbol Device:R
- added RV? (x12): R_POT, Potentiometer_THT:Potentiometer_Alps_RK09K_Single_Vertical, symbol Device:R_POT
- added U?: 4051, Package_SO:SOIC-16_3.9x9.9mm_P1.27mm, symbol 4xxx:4051
- added U?: Teensy4.1, symbol teensy:Teensy4.1
Connections:
- net ANA_CHAN0: now also U?.11 (A)
- net ANA_CHAN1: now also U?.10 (B)
- net ANA_CHAN2: now also U?.9 (C)
- net GND: now also RV?.3, RV?.3, RV?.3, RV?.3, RV?.3, RV?.3, RV?.3, RV?.3, RV?.3, RV?.3, RV?.3, RV?.3, U?.6 (Inh), U?.7 (VEE), U?.8 (VSS); no longer D1.1 (K), D2.1 (K), D3.1 (K), D4.1 (K)
- net POT1: now also RV2.2, U4.14 (X1); no longer RV1.2, U4.13 (X0)
- net POT2: now also RV3.2, U4.15 (X2); no longer RV2.2, U4.14 (X1)
- net POT3: now also RV4.2, U4.12 (X3); no longer RV3.2, U4.15 (X2)
- net POT4: now also U4.1 (X4), RV?.2; no longer RV4.2, U4.12 (X3)
- net VCC: now also RV?.1, RV?.1, RV?.1, RV?.1, RV?.1, RV?.1, RV?.1, RV?.1, RV?.1, RV?.1, RV?.1, RV?.1, U?.16 (VDD)
- net POT6: now reaches U4.2 (X6)
- net POT6: now also RV?.2
- net POT7: now reaches U4.4 (X7)
- net POT7: now also RV?.2
- net POT5: now reaches U4.5 (X5)
- net POT5: now also RV?.2
- net at U3.4 (QE): now also R?.2
- net at U3.5 (QF): now also R?.2
- net at U3.6 (QG): now also R?.2
- net at U3.7 (QH): now also R?.2
- net ANA_OUT renamed ANA_OUT0
- net LED_DATA_OUT: no longer names the net of U3.9 (QH')
- new net: D1.1 (K), D2.1 (K), D3.1 (K), D4.1 (K), D?.1 (K), D?.1 (K), D?.1 (K), D?.1 (K)
- new net: D?.2 (A), R?.1 (x4)
- new net ANA_OUT1: U?.3 (X)
- new net POT0: RV1.2, U4.13 (X0)
- new net POT10: RV?.2, U?.15 (X2)
- new net POT11: RV?.2, U?.12 (X3)
- new net POT12: RV?.2, U?.1 (X4)
- new net POT13: RV?.2, U?.5 (X5)
- new net POT14: RV?.2, U?.2 (X6)
- new net POT15: RV?.2, U?.4 (X7)
- new net POT8: RV?.2, U?.13 (X0)
- new net POT9: RV?.2, U?.14 (X1)
- no-connect marks 14 -> 6
Other:
- moved on the sheet: D1, D2, D3, D4, H1, H2, J?, R1, R10, R11, R12, R13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

Commit message: mini schematic nearly done
Parts:
- added C?: CP, symbol Device:CP
- added D?: 1N4148, Diode_THT:D_DO-35_SOD27_P7.62mm_Horizontal, symbol Diode:1N4148
- added J3: Conn_01x10, symbol Connector_Generic:Conn_01x10
- added J?: DIN-5_180degree, symbol Connector:DIN-5_180degree
- added R? (x2): R, symbol Device:R
- added U?: 6N138, symbol Isolator:6N138
- gave numbers to parts that had none: 62
Connections:
- net ANA_OUT0 is gone; now on net ANA_DATA0: U4.3 (X)
- net ANA_OUT1 is gone; now on net ANA_DATA1: U10.3 (X)
- net IN_DATA_OUT is gone; now on net IN_DATA: U2.10 (DS)
- net LED_DATA_IN is gone; now on net LED_DATA: U3.14 (SER)
- net OUT_DATA_IN is gone; now on net OUT_DATA: U1.14 (SER)
- net ANA_CHAN0: now also U9.16 (24_A10_TX6_SCL2)
- net ANA_CHAN1: now also U9.17 (25_A11_RX6_SDA2)
- net ANA_CHAN2: now also U9.18 (26_A12_MOSI1)
- net GND: now also U9.1 (GND), U9.34 (GND), U9.47 (GND), J3.1 (Pin_1)
- net IN_CLOCK: now also U9.7 (5_IN2)
- net IN_CLOCK_ENABLE: now also U9.8 (6_OUT1D)
- net IN_LOAD: now also U9.11 (9_OUT1C)
- net LED_CLOCK: now also U9.37 (15_A1_RX3_SPDIF_IN)
- net LED_LATCH: now also U9.36 (14_A0_TX3_SPDIF_OUT)
- net OUT_CLOCK: now also U9.4 (2_OUT2)
- net OUT_LATCH: now also U9.5 (3_LRCLK2)
- net VCC: now also U9.15 (3V3)
- net ANA_DATA0: now reaches U9.19 (27_A13_SCK1)
- net MIDI_IN: now reaches U9.2 (0_RX1_CRX2_CS1)
- net ANA_DATA1: now reaches U9.20 (28_RX7)
- net at U9.25 (33_MCLK2): now also J3.10 (Pin_10)
- net at U9.26 (34_RX8): now also J3.9 (Pin_9)
- net at U9.27 (35_TX8): now also J3.8 (Pin_8)
- net at U9.28 (36_CS): now also J3.7 (Pin_7)
- net at U9.29 (37_CS): now also J3.6 (Pin_6)
- net OUT_DATA: now reaches U9.3 (1_TX1_CTX2_MISO1)
- net at U9.30 (38_CS1_IN1): now also J3.5 (Pin_5)
- net at U9.31 (39_MISO1_OUT1A): now also J3.4 (Pin_4)
- net at U9.32 (40_A16): now also J3.3 (Pin_3)
- net at U9.33 (41_A17): now also J3.2 (Pin_2)
- net LED_DATA: now reaches U9.38 (16_A2_RX4_SCL1)
- net IN_DATA: now reaches U9.6 (4_BCLK2)
- no-connect marks 6 -> 44

Commit message: mini pcb layout started
Parts:
- added R59: 470, Resistor_SMD:R_0805_2012Metric, symbol Device:R
- C1: renamed from C?; value CP -> 100nF; footprint (none) -> Resistor_SMD:R_0805_2012Metric
- J1, J2: footprint (none) -> Connector_PinSocket_2.54mm:PinSocket_2x12_P2.54mm_Vertical
- J3: renamed from J?; footprint (none) -> p3mini:MIDI_DIN5
- J4: renamed from J3; footprint (none) -> Connector_PinSocket_2.54mm:PinSocket_1x10_P2.54mm_Vertical
- R1, R2, R3, R4, R5, R6, R7, R8: footprint Resistor_SMD:R_1206_3216Metric -> Resistor_SMD:R_0805_2012Metric
- R10: renamed from R22; footprint Resistor_SMD:R_1206_3216Metric -> Resistor_SMD:R_0805_2012Metric
- R11: renamed from R23; footprint Resistor_SMD:R_1206_3216Metric -> Resistor_SMD:R_0805_2012Metric
- R12: renamed from R24; footprint Resistor_SMD:R_1206_3216Metric -> Resistor_SMD:R_0805_2012Metric
- R13: renamed from R25; footprint Resistor_SMD:R_1206_3216Metric -> Resistor_SMD:R_0805_2012Metric
- R14: renamed from R26; footprint Resistor_SMD:R_1206_3216Metric -> Resistor_SMD:R_0805_2012Metric
- R15: renamed from R27; footprint Resistor_SMD:R_1206_3216Metric -> Resistor_SMD:R_0805_2012Metric
- R16: renamed from R28; footprint Resistor_SMD:R_1206_3216Metric -> Resistor_SMD:R_0805_2012Metric
- R17: renamed from R29; footprint Resistor_SMD:R_1206_3216Metric -> Resistor_SMD:R_0805_2012Metric
- R18: renamed from R30; footprint Resistor_SMD:R_1206_3216Metric -> Resistor_SMD:R_0805_2012Metric
- R19: renamed from R31; footprint Resistor_SMD:R_1206_3216Metric -> Resistor_SMD:R_0805_2012Metric
- R20: renamed from R32; footprint Resistor_SMD:R_1206_3216Metric -> Resistor_SMD:R_0805_2012Metric
- R21: renamed from R33; footprint Resistor_SMD:R_1206_3216Metric -> Resistor_SMD:R_0805_2012Metric
- R22: renamed from R34; footprint Resistor_SMD:R_1206_3216Metric -> Resistor_SMD:R_0805_2012Metric
- R23: renamed from R35; footprint Resistor_SMD:R_1206_3216Metric -> Resistor_SMD:R_0805_2012Metric
- R24: renamed from R36; footprint Resistor_SMD:R_1206_3216Metric -> Resistor_SMD:R_0805_2012Metric
- R25: renamed from R9; footprint Resistor_SMD:R_1206_3216Metric -> Resistor_SMD:R_0805_2012Metric
- R26: renamed from R10; footprint Resistor_SMD:R_1206_3216Metric -> Resistor_SMD:R_0805_2012Metric
- R27: renamed from R11; footprint Resistor_SMD:R_1206_3216Metric -> Resistor_SMD:R_0805_2012Metric
- R28: renamed from R12; footprint Resistor_SMD:R_1206_3216Metric -> Resistor_SMD:R_0805_2012Metric
- R29: renamed from R13; footprint Resistor_SMD:R_1206_3216Metric -> Resistor_SMD:R_0805_2012Metric
- R30: renamed from R14; footprint Resistor_SMD:R_1206_3216Metric -> Resistor_SMD:R_0805_2012Metric
- R31: renamed from R15; footprint Resistor_SMD:R_1206_3216Metric -> Resistor_SMD:R_0805_2012Metric
- R32: renamed from R16; footprint Resistor_SMD:R_1206_3216Metric -> Resistor_SMD:R_0805_2012Metric
- R33: renamed from R37; footprint Resistor_SMD:R_1206_3216Metric -> Resistor_SMD:R_0805_2012Metric
- R34: renamed from R38; footprint Resistor_SMD:R_1206_3216Metric -> Resistor_SMD:R_0805_2012Metric
- R35: renamed from R39; footprint Resistor_SMD:R_1206_3216Metric -> Resistor_SMD:R_0805_2012Metric
- R36: renamed from R40; footprint Resistor_SMD:R_1206_3216Metric -> Resistor_SMD:R_0805_2012Metric
- R37: renamed from R41; footprint Resistor_SMD:R_1206_3216Metric -> Resistor_SMD:R_0805_2012Metric
- R38: renamed from R42; footprint Resistor_SMD:R_1206_3216Metric -> Resistor_SMD:R_0805_2012Metric
- R39: renamed from R43; footprint Resistor_SMD:R_1206_3216Metric -> Resistor_SMD:R_0805_2012Metric
- R40: renamed from R44; footprint Resistor_SMD:R_1206_3216Metric -> Resistor_SMD:R_0805_2012Metric
- R41: renamed from R45; footprint Resistor_SMD:R_1206_3216Metric -> Resistor_SMD:R_0805_2012Metric
- R42: renamed from R46; footprint Resistor_SMD:R_1206_3216Metric -> Resistor_SMD:R_0805_2012Metric
- R43: renamed from R47; footprint Resistor_SMD:R_1206_3216Metric -> Resistor_SMD:R_0805_2012Metric
- R44: renamed from R48; footprint Resistor_SMD:R_1206_3216Metric -> Resistor_SMD:R_0805_2012Metric
- R45: renamed from R49; footprint Resistor_SMD:R_1206_3216Metric -> Resistor_SMD:R_0805_2012Metric
- R46: renamed from R50; footprint Resistor_SMD:R_1206_3216Metric -> Resistor_SMD:R_0805_2012Metric
- R47: renamed from R51; footprint Resistor_SMD:R_1206_3216Metric -> Resistor_SMD:R_0805_2012Metric
- R48: renamed from R52; footprint Resistor_SMD:R_1206_3216Metric -> Resistor_SMD:R_0805_2012Metric
- R57: renamed from R?; value R -> 220; footprint (none) -> Resistor_SMD:R_1206_3216Metric
- R58: renamed from R?; value R -> 10k; footprint (none) -> Resistor_SMD:R_0805_2012Metric
- R9: renamed from R21; footprint Resistor_SMD:R_1206_3216Metric -> Resistor_SMD:R_0805_2012Metric
- RV1, RV11, RV12, RV13, RV14, RV15, RV16: footprint Potentiometer_THT:Potentiometer_Alps_RK09K_Single_Vertical -> p3mini:Potentiometer_Alps_RK09K_Single_Vertical
- RV10: renamed from RV4; footprint Potentiometer_THT:Potentiometer_Alps_RK09K_Single_Vertical -> p3mini:Potentiometer_Alps_RK09K_Single_Vertical
- RV2: renamed from RV5; footprint Potentiometer_THT:Potentiometer_Alps_RK09K_Single_Vertical -> p3mini:Potentiometer_Alps_RK09K_Single_Vertical
- RV3: renamed from RV6; footprint Potentiometer_THT:Potentiometer_Alps_RK09K_Single_Vertical -> p3mini:Potentiometer_Alps_RK09K_Single_Vertical
- RV4: renamed from RV2; footprint Potentiometer_THT:Potentiometer_Alps_RK09K_Single_Vertical -> p3mini:Potentiometer_Alps_RK09K_Single_Vertical
- RV5: renamed from RV7; footprint Potentiometer_THT:Potentiometer_Alps_RK09K_Single_Vertical -> p3mini:Potentiometer_Alps_RK09K_Single_Vertical
- RV6: renamed from RV8; footprint Potentiometer_THT:Potentiometer_Alps_RK09K_Single_Vertical -> p3mini:Potentiometer_Alps_RK09K_Single_Vertical
- RV7: renamed from RV3; footprint Potentiometer_THT:Potentiometer_Alps_RK09K_Single_Vertical -> p3mini:Potentiometer_Alps_RK09K_Single_Vertical
- RV8: renamed from RV9; footprint Potentiometer_THT:Potentiometer_Alps_RK09K_Single_Vertical -> p3mini:Potentiometer_Alps_RK09K_Single_Vertical
- RV9: renamed from RV10; footprint Potentiometer_THT:Potentiometer_Alps_RK09K_Single_Vertical -> p3mini:Potentiometer_Alps_RK09K_Single_Vertical
- U8: renamed from U9; footprint (none) -> teensy:Teensy41
- U9: renamed from U?; footprint (none) -> Package_SO:SSO-8_6.7x9.8mm_P2.54mm_Clearance8mm
- gave numbers to parts that had none: 1
- renumbered R17 to R49, R18 to R50, R19 to R51, R20 to R52, U4 to U10, U10 to U11, U5 to U2, U6 to U3, U2 to U4, U7 to U5, U8 to U6, U3 to U7
Connections:
- net GND: now also C1.2, R58.1, U9.5 (GND)
- net MIDI_IN: now also U9.6 (VO2), R59.2
- net VCC: now also C1.1, U9.8 (VCC), R59.1
- net at U9.2 (C1): now also D9.1 (K), R57.1
- net at U9.3 (C2): now also D9.2 (A), J3.5
- net at U9.7 (VO1): now also R58.2
- net at R57.2: now also J3.4
- no-connect marks 44 -> 47
Other:
- moved on the sheet: C1, D9, J3, R57, R58, U10, U11, U9

Commit message: layout
Parts:
- D9: footprint Diode_THT:D_DO-35_SOD27_P7.62mm_Horizontal -> Diode_SMD:D_SOD-123
- renumbered RV11 to RV10, RV14 to RV11, RV16 to RV12, RV3 to RV13, RV6 to RV14, RV9 to RV15, RV12 to RV16, RV4 to RV2, RV7 to RV3, RV10 to RV4, RV13 to RV5, RV15 to RV6, RV2 to RV7, RV5 to RV8, RV8 to RV9
Connections:
- net INPUT1: now also J2.3 (Pin_3); no longer J2.2 (Pin_2)
- net INPUT10: now also J2.21 (Pin_21); no longer J2.11 (Pin_11)
- net INPUT11: now also J2.23 (Pin_23); no longer J2.12 (Pin_12)
- net INPUT12: now also J2.24 (Pin_24); no longer J2.13 (Pin_13)
- net INPUT13: now also J2.22 (Pin_22); no longer J2.14 (Pin_14)
- net INPUT14: now also J2.20 (Pin_20); no longer J2.15 (Pin_15)
- net INPUT15: now also J2.18 (Pin_18); no longer J2.16 (Pin_16)
- net INPUT16: now also J2.16 (Pin_16); no longer J2.17 (Pin_17)
- net INPUT17: now also J2.14 (Pin_14); no longer J2.18 (Pin_18)
- net INPUT18: now also J2.12 (Pin_12); no longer J2.19 (Pin_19)
- net INPUT19: now also J2.10 (Pin_10); no longer J2.20 (Pin_20)
- net INPUT2: now also J2.5 (Pin_5); no longer J2.3 (Pin_3)
- net INPUT20: now also J2.8 (Pin_8); no longer J2.21 (Pin_21)
- net INPUT21: now also J2.6 (Pin_6); no longer J2.22 (Pin_22)
- net INPUT22: now also J2.4 (Pin_4); no longer J2.23 (Pin_23)
- net INPUT23: now also J2.2 (Pin_2); no longer J2.24 (Pin_24)
- net INPUT3: now also J2.7 (Pin_7); no longer J2.4 (Pin_4)
- net INPUT4: now also J2.9 (Pin_9); no longer J2.5 (Pin_5)
- net INPUT5: now also J2.11 (Pin_11); no longer J2.6 (Pin_6)
- net INPUT6: now also J2.13 (Pin_13); no longer J2.7 (Pin_7)
- net INPUT7: now also J2.15 (Pin_15); no longer J2.8 (Pin_8)
- net INPUT8: now also J2.17 (Pin_17); no longer J2.9 (Pin_9)
- net INPUT9: now also J2.19 (Pin_19); no longer J2.10 (Pin_10)
- net OUTPUT1: now also J1.3 (Pin_3); no longer J1.2 (Pin_2)
- net OUTPUT10: now also J1.21 (Pin_21); no longer J1.11 (Pin_11)
- net OUTPUT11: now also J1.23 (Pin_23); no longer J1.12 (Pin_12)
- net OUTPUT12: now also J1.24 (Pin_24); no longer J1.13 (Pin_13)
- net OUTPUT13: now also J1.22 (Pin_22); no longer J1.14 (Pin_14)
- net OUTPUT14: now also J1.20 (Pin_20); no longer J1.15 (Pin_15)
- net OUTPUT15: now also J1.18 (Pin_18); no longer J1.16 (Pin_16)
- net OUTPUT16: now also J1.16 (Pin_16); no longer J1.17 (Pin_17)
- net OUTPUT17: now also J1.14 (Pin_14); no longer J1.18 (Pin_18)
- net OUTPUT18: now also J1.12 (Pin_12); no longer J1.19 (Pin_19)
- net OUTPUT19: now also J1.10 (Pin_10); no longer J1.20 (Pin_20)
- net OUTPUT2: now also J1.5 (Pin_5); no longer J1.3 (Pin_3)
- net OUTPUT20: now also J1.8 (Pin_8); no longer J1.21 (Pin_21)
- net OUTPUT21: now also J1.6 (Pin_6); no longer J1.22 (Pin_22)
- net OUTPUT22: now also J1.4 (Pin_4); no longer J1.23 (Pin_23)
- net OUTPUT23: now also J1.2 (Pin_2); no longer J1.24 (Pin_24)
- net OUTPUT3: now also J1.7 (Pin_7); no longer J1.4 (Pin_4)
- net OUTPUT4: now also J1.9 (Pin_9); no longer J1.5 (Pin_5)
- net OUTPUT5: now also J1.11 (Pin_11); no longer J1.6 (Pin_6)
- net OUTPUT6: now also J1.13 (Pin_13); no longer J1.7 (Pin_7)
- net OUTPUT7: now also J1.15 (Pin_15); no longer J1.8 (Pin_8)
- net OUTPUT8: now also J1.17 (Pin_17); no longer J1.9 (Pin_9)
- net OUTPUT9: now also J1.19 (Pin_19); no longer J1.10 (Pin_10)
